Commit message: 241203

File: urdf_tutorial/urdf/robot_1.xacro (robot description, xacro)
@@ -1,4 +1,4 @@
 <?xmal version="1.0"?>
-<robot xmls:xacro='https://ros.org/wikiu/xacro' name='urdf_test'>
+<robot xmlns:xacro='https://ros.org/wiki/xacro' name='urdf_test'>
     <link name = 'base_link'>
     </link>
@@ -10,5 +10,5 @@
         <visual>
             <geometry>
-                <box size = '1 1 1'/>
+                <box size ='1 1 1'/>
             </geometry>
         </visual>
