Commit message: 241203_2

File: description/urdf/robot_2.xacro (robot description, xacro)
@@ -10,5 +10,5 @@
             <origin rpy="0.0 0 0" xyz="0 0 0"/>
             <geometry>
-                <mesh filename="package://urdf_tutorial/meshes/aaa.stl" scale="1 1 1"/>
+                <mesh filename="package://description/meshes/aaa.stl" scale="1 1 1"/>
             </geometry>
         </visual>

Commit message: 241203

File: description/urdf/robot_2.xacro (robot description, xacro)
@@ -1,23 +1,33 @@
 <?xmal version="1.0"?>
 <robot xmlns:xacro='https://ros.org/wiki/xacro' name='urdf_test'>
+    <xacro:property name="wheel_diameter" value="0.068"/>
+    <xacro:property name="wheel_speration" value="0.180"/>
     <link name = 'base_link'/>
     <joint name = 'body_joint' type='fixed'>
         <parent link='base_link'/>
-        <child link = 'test'/>
+        <child link = 'robot_body'/>
+        <origin xyz="0.129 0.0 0.0" rpy="0.0 0.0 0.0"/>
     </joint>
-    <link name="test">
+    <link name="robot_body">
         <visual>
-            <origin rpy="0.0 0 0" xyz="0 0 0"/>
+            <origin rpy="0 0 0" xyz="0 0 0"/>
             <geometry>
-                <mesh filename="package://description/meshes/aaa.stl" scale="1 1 1"/>
+                <mesh filename="package://description/meshes/base.stl" scale="0.001 0.001 0.001"/>
             </geometry>
         </visual>
     </link>
-    <!--<link name = 'body'>
+    <joint name="r_wheel_joint" type="continuous">
+        <parent link='robot_body'/>
+        <child link='r_wheel'/>
+        <origin xyz="0.129 0.0 0.0" rpy="0.0 0.0 0.0"/>
+        <axis xyz="0 1 0"/>
+    </joint>
+    <link name="r_wheel">
         <visual>
+            <origin rpy="0 0 0" xyz="0 0 0"/>
             <geometry>
-                <box size ='1 1 1'/>
+                <mesh filename="package://description/meshes/wheel.stl" scale="0.001 0.001 0.001"/>
             </geometry>
         </visual>
-    </link>-->
+    </link>
 </robot>

Commit message: 241204

File: description/urdf/robot_2.xacro (robot description, xacro)
@@ -3,4 +3,7 @@
     <xacro:property name="wheel_diameter" value="0.068"/>
     <xacro:property name="wheel_speration" value="0.180"/>
+    <material name="white">
+        <color rgba="1 1 1 1" />
+    </material>
     <link name = 'base_link'/>
     <joint name = 'body_joint' type='fixed'>
@@ -11,23 +14,45 @@
     <link name="robot_body">
         <visual>
-            <origin rpy="0 0 0" xyz="0 0 0"/>
+            <origin xyz="0 0 0" rpy="0 0 0"/>
             <geometry>
-                <mesh filename="package://description/meshes/base.stl" scale="0.001 0.001 0.001"/>
+                <mesh filename="package://description/meshes/robot_b_body.stl" scale="0.001 0.001 0.001"/>
             </geometry>
+            <material name="white"/>
         </visual>
     </link>
+    <!-- <gazebo reference='robot_body'>
+        <material>Gazebo/White</material>
+    </gazebo> -->
     <joint name="r_wheel_joint" type="continuous">
         <parent link='robot_body'/>
         <child link='r_wheel'/>
-        <origin xyz="0.129 0.0 0.0" rpy="0.0 0.0 0.0"/>
+        <origin xyz="0.0 0.0 0.0" rpy="0.0 0.0 0.0"/>
         <axis xyz="0 1 0"/>
     </joint>
     <link name="r_wheel">
         <visual>
-            <origin rpy="0 0 0" xyz="0 0 0"/>
+            <origin xyz="0 0 0" rpy="0 0 0"/>
             <geometry>
-                <mesh filename="package://description/meshes/wheel.stl" scale="0.001 0.001 0.001"/>
+                <mesh filename="package://description/meshes/robot_b_r_wheel.stl" scale="0.001 0.001 0.001"/>
             </geometry>
         </visual>
     </link>
+    <!-- <gazebo reference='r_wheel'>
+        <material>Gazebo/Black</material>
+    </gazebo> -->
+    <joint name="l_wheel_joint" type="continuous">
+        <parent link="robot_body"/>
+        <child link="l_wheel"/>
+    </joint>
+    <link name="l_wheel">
+        <visual>
+            <origin xyz="0 0 0 " rpy=" 0 0 0"/>
+                <geometry>
+                    <mesh filename="package://description/meshes/robot_b_l_wheel.stl" scale="0.001 0.001 0.001"/>
+                </geometry>
+        </visual>
+    </link>
+    <!-- <gazebo reference='l_wheel'>
+        <material>Gazebo/Black</material>
+    </gazebo> -->
 </robot>

Commit message: 241204_2

File: description/urdf/robot_2.xacro (robot description, xacro)
@@ -10,5 +10,5 @@
         <parent link='base_link'/>
         <child link = 'robot_body'/>
-        <origin xyz="0.129 0.0 0.0" rpy="0.0 0.0 0.0"/>
+        <origin xyz="0.0 0.0 0.0" rpy="0.0 0.0 0.0"/>
     </joint>
     <link name="robot_body">
@@ -16,5 +16,5 @@
             <origin xyz="0 0 0" rpy="0 0 0"/>
             <geometry>
-                <mesh filename="package://description/meshes/robot_b_body.stl" scale="0.001 0.001 0.001"/>
+                <mesh filename="package://description/meshes/robot_b_all.stl" scale="0.001 0.001 0.001"/>
             </geometry>
             <material name="white"/>

Commit message: 241204_2

File: description/urdf/robot_2.xacro (robot description, xacro)
@@ -16,5 +16,5 @@
             <origin xyz="0 0 0" rpy="0 0 0"/>
             <geometry>
-                <mesh filename="package://description/meshes/robot_b_all.stl" scale="0.001 0.001 0.001"/>
+                <mesh filename="package://description/meshes/robot_a/robot_a_body2.stl" scale="0.001 0.001 0.001"/>
             </geometry>
             <material name="white"/>
@@ -27,12 +27,11 @@
         <parent link='robot_body'/>
         <child link='r_wheel'/>
-        <origin xyz="0.0 0.0 0.0" rpy="0.0 0.0 0.0"/>
-        <axis xyz="0 1 0"/>
+        <origin xyz="0.1 0.168 0.168" rpy="0.0 0.0 3.14"/>
     </joint>
     <link name="r_wheel">
         <visual>
-            <origin xyz="0 0 0" rpy="0 0 0"/>
+            <origin xyz="-0.05 -0.168 -0.168" rpy="0 0 0"/>
             <geometry>
-                <mesh filename="package://description/meshes/robot_b_r_wheel.stl" scale="0.001 0.001 0.001"/>
+                <mesh filename="package://description/meshes/robot_b/robot_b_r_wheel.stl" scale="0.001 0.001 0.001"/>
             </geometry>
         </visual>
@@ -42,4 +41,5 @@
     </gazebo> -->
     <joint name="l_wheel_joint" type="continuous">
+        <origin xyz="0.50 0.168 0.168" rpy="0 0 0"/>
         <parent link="robot_body"/>
         <child link="l_wheel"/>
@@ -47,7 +47,7 @@
     <link name="l_wheel">
         <visual>
-            <origin xyz="0 0 0 " rpy=" 0 0 0"/>
+            <origin xyz="-0.04 -0.168 -0.168" rpy=" 0 0 0"/>
                 <geometry>
-                    <mesh filename="package://description/meshes/robot_b_l_wheel.stl" scale="0.001 0.001 0.001"/>
+                    <mesh filename="package://description/meshes/robot_b/robot_b_l_wheel.stl" scale="0.001 0.001 0.001"/>
                 </geometry>
         </visual>

Commit message: 241204_3

File: description/urdf/robot_2.xacro (robot description, xacro)
@@ -16,5 +16,5 @@
             <origin xyz="0 0 0" rpy="0 0 0"/>
             <geometry>
-                <mesh filename="package://description/meshes/robot_a/robot_a_body2.stl" scale="0.001 0.001 0.001"/>
+                <mesh filename="package://description/meshes/robot_b/robot_b_body.stl" scale="0.001 0.001 0.001"/>
             </geometry>
             <material name="white"/>
@@ -26,12 +26,13 @@
     <joint name="r_wheel_joint" type="continuous">
         <parent link='robot_body'/>
-        <child link='r_wheel'/>
-        <origin xyz="0.1 0.168 0.168" rpy="0.0 0.0 3.14"/>
+        <child link='r_wheel'/>0
+        <origin xyz="0.05 0.168 0.168" rpy="0 -1.57 0"/>
+        <axis xyz='0 0 1'/>
     </joint>
     <link name="r_wheel">
         <visual>
-            <origin xyz="-0.05 -0.168 -0.168" rpy="0 0 0"/>
+            <origin xyz="-0.168 -0.168 0.04" rpy="0 1.57 0"/>
             <geometry>
-                <mesh filename="package://description/meshes/robot_b/robot_b_r_wheel.stl" scale="0.001 0.001 0.001"/>
+                <mesh filename="package://description/meshes/robot_b/robot_b_l_wheel.stl" scale="0.001 0.001 0.001"/>
             </geometry>
         </visual>

Commit message: 241204_3

File: description/urdf/robot_2.xacro (robot description, xacro)
@@ -32,7 +32,7 @@
     <link name="r_wheel">
         <visual>
-            <origin xyz="-0.168 -0.168 0.04" rpy="0 1.57 0"/>
+            <origin xyz="-0.168 -0.168 0.05" rpy="0 1.57 0"/>
             <geometry>
-                <mesh filename="package://description/meshes/robot_b/robot_b_l_wheel.stl" scale="0.001 0.001 0.001"/>
+                <mesh filename="package://description/meshes/robot_b/robot_b_r_wheel.stl" scale="0.001 0.001 0.001"/>
             </geometry>
         </visual>
@@ -42,11 +42,12 @@
     </gazebo> -->
     <joint name="l_wheel_joint" type="continuous">
-        <origin xyz="0.50 0.168 0.168" rpy="0 0 0"/>
+        <origin xyz="0.50 0.168 0.168" rpy="0 1.57 0"/>
         <parent link="robot_body"/>
         <child link="l_wheel"/>
+        <axis xyz='0 0 1'/>
     </joint>
     <link name="l_wheel">
         <visual>
-            <origin xyz="-0.04 -0.168 -0.168" rpy=" 0 0 0"/>
+            <origin xyz="0.17 -0.16 -0.038" rpy="0 -1.57 0"/>
                 <geometry>
                     <mesh filename="package://description/meshes/robot_b/robot_b_l_wheel.stl" scale="0.001 0.001 0.001"/>
