Commit message: 241204

File: description/urdf/robot_1.xacro (robot description, xacro)
@@ -10,9 +10,9 @@
         <parent link='base_link'/>
         <child link = 'robot_body'/>
-        <origin xyz="0.0 0.0 0.0" rpy="0.0 0.0 0.0"/>
+        <origin xyz="0.0 0.0 0.36" rpy="0.0 0.0 0.0"/>
     </joint>
     <link name="robot_body">
         <visual>
-            <origin xyz="0 0 0" rpy="0 0 0"/>
+            <origin xyz="0.0 0.0 0.0" rpy="0 0 0.0"/>
             <geometry>
                 <mesh filename="package://description/meshes/robot_a/robot_a_body.stl" scale="0.001 0.001 0.001"/>
@@ -27,10 +27,10 @@
         <parent link='robot_body'/>
         <child link='r_wheel'/>
-        <origin xyz="0.05 0.168 0.168" rpy="0 -1.57 0"/>
+        <origin xyz="0.35 -0.23 -0.23" rpy="1.57 0 0"/>
         <axis xyz='0 0 1'/>
     </joint>
     <link name="r_wheel">
         <visual>
-            <origin xyz="-0.168 -0.168 0.05" rpy="0 1.57 0"/>
+            <origin xyz="0 0 0" rpy="0 0 0"/>
             <geometry>
                 <mesh filename="package://description/meshes/robot_a/robot_a_r_wheel.stl" scale="0.001 0.001 0.001"/>
@@ -42,5 +42,5 @@
     </gazebo> -->
     <joint name="l_wheel_joint" type="continuous">
-        <origin xyz="0.50 0.168 0.168" rpy="0 1.57 0"/>
+        <origin xyz="0.35 0.23 -0.23" rpy="-1.57 0 0"/>
         <parent link="robot_body"/>
         <child link="l_wheel"/>
@@ -49,5 +49,5 @@
     <link name="l_wheel">
         <visual>
-            <origin xyz="0.17 -0.16 -0.038" rpy="0 -1.57 0"/>
+            <origin xyz="0 0 0" rpy="0 0 0"/>
                 <geometry>
                     <mesh filename="package://description/meshes/robot_a/robot_a_l_wheel.stl" scale="0.001 0.001 0.001"/>

File: description/urdf/robot_2.xacro (robot description, xacro)
@@ -27,10 +27,10 @@
         <parent link='robot_body'/>
         <child link='r_wheel'/>0
-        <origin xyz="0.05 0.168 0.168" rpy="0 -1.57 0"/>
+        <origin xyz="0.0 0.0 0.0" rpy="0 0 0"/>
         <axis xyz='0 0 1'/>
     </joint>
     <link name="r_wheel">
         <visual>
-            <origin xyz="-0.168 -0.168 0.05" rpy="0 1.57 0"/>
+            <origin xyz="0.0 0.0 0.0" rpy="0 0 0"/>
             <geometry>
                 <mesh filename="package://description/meshes/robot_b/robot_b_r_wheel.stl" scale="0.001 0.001 0.001"/>
@@ -42,5 +42,5 @@
     </gazebo> -->
     <joint name="l_wheel_joint" type="continuous">
-        <origin xyz="0.50 0.168 0.168" rpy="0 1.57 0"/>
+        <origin xyz="0.0 0.0 0.0" rpy="0 0 0"/>
         <parent link="robot_body"/>
         <child link="l_wheel"/>
@@ -49,5 +49,5 @@
     <link name="l_wheel">
         <visual>
-            <origin xyz="0.17 -0.16 -0.038" rpy="0 -1.57 0"/>
+            <origin xyz="0.0 0.0 0.0" rpy="0 0 0"/>
                 <geometry>
                     <mesh filename="package://description/meshes/robot_b/robot_b_l_wheel.stl" scale="0.001 0.001 0.001"/>
